Commit message: Fix URDF

File: src/hamster_simulation/hamster_vehicle_description/urdf/hamster.urdf.xacro (robot description, xacro)
@@ -11,10 +11,11 @@
   <xacro:arg name="robot_version" default="V6"/>
   <xacro:property name="version" value="$(arg robot_version)"/>
-  <link name="dummy"></link>
-  <link name="base_link">
+  <link name="dummy">
     <inertial>
       <mass value="3.0" />
       <inertia ixx="0.025" iyy="0.025" izz="5e-3" ixy="0" iyz="0" ixz="0"/>
     </inertial>
+  </link>
+  <link name="base_link">
     <visual>
       <geometry>
@@ -29,6 +30,6 @@
   </link>
   <joint name="dummy_joint" type="fixed">
-     <parent link="dummy"/>
-     <child link="base_link"/>
+     <parent link="base_link"/>
+     <child link="dummy"/>
    </joint>
   <link name="imu_link">

Commit message: fixed: incorrect laser name

File: src/hamster_simulation/hamster_vehicle_description/urdf/hamster.urdf.xacro (robot description, xacro)
@@ -44,9 +44,4 @@
     </visual>
     </link>
-  <!-- <joint name="dummy_link_joint" type="fixed">
-    <origin xyz="0 0 0" rpy="0 0 0" />
-    <parent link="dummy" />
-    <child  link="base_link" />
-  </joint> -->
   <joint name="imu_link_joint" type="fixed">
     <origin xyz="0 0 0" rpy="0 0 0" />
@@ -167,5 +162,5 @@
     <sensor type="gpu_ray" name="head_hokuyo_sensor">
       <pose>0 0 0 0 0 0</pose>
-      <visualize>false</visualize>
+      <visualize>true</visualize>
       <update_rate>10</update_rate>
       <ray>
@@ -191,5 +186,5 @@
       <plugin name="gazebo_ros_head_hokuyo_controller" filename="libgazebo_ros_gpu_laser.so">
         <topicName>scan</topicName>
-        <frameName>lidar_link</frameName>
+        <frameName>$(arg agent)/lidar_link</frameName>
       </plugin>
     </sensor>
